File: schematic/schematic.kicad_sch (KiCad schematic)
At the start: 0 parts

Commit message: created clock sheet, added LM555 timers
Other:
- added sheet clock (clock_sch.kicad_sch)
Changed lines of the file:
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@@
 (kicad_sch (version 20211123) (generator eeschema)
   (paper "A4")
+  (sheet (at 25.4 25.4) (size 40.64 34.29) (fields_autoplaced)
+    (stroke (width 0.1524) (type solid) (color 0 0 0 0))
+    (fill (color 0 0 0 0.0000))
+    (property "Sheet name" "clock" (id 0) (at 25.4 24.6884 0)
+      (effects (font (size 1.27 1.27)) (justify left bottom))
+    )
+    (property "Sheet file" "clock_sch.kicad_sch" (id 1) (at 25.4 60.2746 0)
+      (effects (font (size 1.27 1.27)) (justify left top))
+    )
+  )
   (sheet_instances
     (path "/" (page "1"))
+    (path "/f381231e-3904-4cea-bcb9-dd8495327832" (page "2"))
+  )
+  (symbol_instances
+    (path "/f381231e-3904-4cea-bcb9-dd8495327832/271bcbd5-d434-4876-b051-ba7ac054d787"
+      (reference "U?") (unit 1) (value "LM555xM") (footprint "Package_SO:SOIC-8_3.9x4.9mm_P1.27mm")
+    )
+    (path "/f381231e-3904-4cea-bcb9-dd8495327832/33147ef2-4c9c-491b-9000-e3e0dcf4d4fd"
+      (reference "U?") (unit 1) (value "LM555xM") (footprint "Package_SO:SOIC-8_3.9x4.9mm_P1.27mm")
+    )
+    (path "/f381231e-3904-4cea-bcb9-dd8495327832/3c812e3d-2d08-4318-8943-b717d4d7431c"
+      (reference "U?") (unit 1) (value "LM555xM") (footprint "Package_SO:SOIC-8_3.9x4.9mm_P1.27mm")
+    )
   )
 )
